File: DC-DC_Converter_RF-15A.kicad_sch (KiCad schematic)
At the start: 73 parts, among them K1 G5L-SMALL, Q1 75NF75_TO-220, Q2 75NF75_TO-220, Q3 NPN_SOT23-3_BEC, Q4 NPN_SOT23-3_BEC, Q5 PNP_SOT-223_BCE, Q6 PNP_SOT-223_BCE, U1 TL494

Commit message: Se termina la PCB, queda acomodar el esquemático
Parts:
- removed C10: C_Axial, Capacitor_THT:CP_Radial_D13.0mm_P7.50mm, symbol 1-Capacitor:C_0805
- removed D8: 1N4148W, Diode_SMD:D_SOD-123, symbol Diode:1N4148W
- added C9: C_Polarized_US, Capacitor_THT:CP_Radial_D13.0mm_P7.50mm, symbol Device:C_Polarized_US
- added D13: BZD27Cxx, Diode_SMD:D_SMF, symbol Diode:BZD27Cxx
- added PAD1, PAD2, PAD3, PAD4: PAD_2.0_1.1, 1-Pad:PAD_2.0_1.1, symbol 1-Pad:PAD_2.0_1.1
- added Q7: PXT2222A_SOT-89, 1-Package_TO_SOT_SMD:SOT-89-3, symbol 1-Transistor:PXT2222A_SOT-89
- C16: footprint Capacitor_THT:CP_Radial_D6.3mm_P2.50mm -> Capacitor_THT:CP_Radial_D5.0mm_P2.50mm
Connections:
- net +BATT: now also R5.1, PAD3.1
- net FB: now also C4.2
- net GND: now also C13.2, C17.2, C2.1, C21.2, C6.2, C7.1, C8.2, D1.2 (A), D10.1 (A), D10.3 (A), D11.K, D9.1 (A), D9.3 (A), Q6.3 (C), R2.1, R22.2, R29.2, RV1.1, U1.10 (E2), U1.13 (OUTCTRL), U1.7 (GND), U1.9 (E1), C9.2, PAD2.1, PAD4.1, Q7.3 (E); no longer RV1.3
- net IN1+: now also R6.2, R7.1
- net IN1-: no longer R6.2, R7.1
- net IN2+: now also C2.2, C3.1, R2.2, R9.2
- net IN2-: now also C3.2, C4.1, C6.1, R28.1, R3.2, R4.2
- net REF: now reaches C12.1, R19.2, R27.2
- net REF: now also U1.14 (REF)
- net VCC: now reaches C21.1
- net VCC: now also R1.2, U1.12 (VCC)
- net +VSW: now reaches R4.1
- net +VSW: now also C20.1, D3.2 (A), K1.S, Q1.2 (D), Q2.2 (D), R1.1, R20.1, R9.1, C9.1
- net at C16.1: now also C18.2, D2.1 (K), Q5.2 (E), R12.2, R13.2, R14.2
- net L2: now reaches C16.2
- net L2: now also C17.1, D10.2 (K), D2.2 (A), D9.2 (K), L1.1, Q1.3 (S), Q2.3 (S)
- net at Q1.1 (G): now also R8.2
- net at D3.1 (K): now also C18.1, R13.1
- net at R3.1: now also Q6.2 (E)
- net at C13.1, D7.1 (K), R25.1: now also R22.1, R32.2; no longer R32.1
- net at D6.1 (K), R25.2: no longer C13.2
- net at R23.2: now also R17.2, D13.1 (K); no longer D7.2 (A)
- net at Q3.1 (B): now also R32.1; no longer R32.2
- net at Q6.1 (B): now also C20.2, C7.2, R20.2, R5.2
- net at R7.2, RV1.2: now also RV1.3; no longer RV1.1
- net at Q5.1 (B): now also R12.1, R15.1
- net at Q5.3 (C): now also R21.2
- net at Q2.1 (G): now also R33.2
- net at R8.1: now also R21.1, R33.1, Q7.2 (C)
- net at C8.1: now also D1.1 (K), R16.1, Q7.1 (B)
- net C2: now reaches R16.2
- net C2: now also R14.1, U1.11 (C2)
- net C1: now reaches R15.2
- net C1: now also U1.8 (C1)
- net at D4.1 (K), D5.1 (K), R30.1: now also K1.2, R31.1
- net VBUS: now reaches D5.2 (A)
- net VBUS: now also K1.P, PAD1.1
- net at Q4.3 (C): now also D4.2 (A), D6.2 (A), K1.1; no longer K1.2
- net at R28.2: now also R29.1
- net at R31.2: now also D11.A
- new net: D13.2 (A), D7.2 (A)
- no-connect marks 0 -> 1
Other:
- moved on the sheet: C1, C11, C12, C13, C16, C17, C18, C19, C2, C20, C21, C3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

Commit message: Se añadieron los valores de algunos componentes, falta ordenar
Parts:
- removed U1: TL494, 1-Package_SO:SOIC-16_4.55x10.3mm_P1.27mm, symbol Regulator_Controller:TL494
- added U2: TL494_SOIC-16, 1-Package_SO:SOIC-16_4.55x10.3mm_P1.27mm, symbol 1-IC-Regulator:TL494_SOIC-16
- C11, C19: value C_Polarized_US -> 2200uF 16V
- C17: value rect -> 1nF 100V
- C18: value rect -> 100nF
- R1: value R_0805 -> 560R
- R10: value R_0805 -> 1M
- R11: value R_0805 -> 47k
- R12, R14, R16, R18, R20, R22, R23, R30, R32, R6: value R_0805 -> 10k
- R15, R3: value R_0805 -> 5.1k
- R17: value R_0805 -> 6.2k
- R19: value R_0805 -> 75k
- R2, R28, R4, R9: value R_0805 -> 100k
- R21, R33, R8: value R_0805 -> 100R
- R24, R29, R5: value R_0805 -> 3.3k
- R25: value R_0805 -> 22k
- R26: value R_0805 -> 39k
- R27, R31: value R_0805 -> 4.7k
- R7: value R_0805 -> 5.6k
- RV1: value R_Potentiometer -> 2k
- renumbered R13 to 470R1
Connections:
- net C1: now also U2.8 (C1)
- net C2: now also U2.11 (C2)
- net FB: now also U2.3 (FB)
- net GND: now also U2.10 (E2), U2.13 (OUTCTRL), U2.7 (GND), U2.9 (E1)
- net IN1-: now also U2.2 (1IN-)
- net IN2+: now also U2.16 (2IN+)
- net IN2-: now also U2.15 (2IN-)
- net VCC: now also U2.12 (VCC)
- net at C1.1: now also U2.5 (CT)
- net at C12.2, R18.1, R19.1: now also U2.4 (DTC)
- net at R26.1: now also U2.6 (RT)
- net IN1+: no longer names the net of R6.2, R7.1
- net IN1+: now also U2.1 (1IN+)
- net REF renamed +5V
- net +5V: now also U2.14 (REF)
Other:
- note added: "12V"
- note added: "5V"
- note added: "Single-Ended Parallel"
- moved on the sheet: C1, C12, C13, C17, C2, C20, C21, C3, C4, C5, C6, C7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
